File: hardware/otros/pcf1306p/pcf1306p-SMD.brd (EAGLE design)
At the start: 18.8 x 49 mm, 12 parts, among them IC23 74LS32D, IC24 74LS00D, IC25 74*157, IC26 74*157, IC3 74*157, IC4 74*157

Commit message: Roto 90 grados el diseño
Parts:
- moved IC23 47.3 mm to (42.9, 9.05), turned to 90 degrees
- moved IC24 47.3 mm to (42.9, 9.05), turned to 90 degrees
- moved C3 39.9 mm to (37.6, 9.53), turned to 90 degrees
- moved C4 38.5 mm to (36.4, 5.24), turned to 90 degrees
- moved IC26 26.4 mm to (28.1, 9.05), turned to 270 degrees
- moved IC4 26.4 mm to (28.1, 9.05), turned to 90 degrees
- moved JP2 23.8 mm to (24.4, 1.75), turned to 0 degrees
- moved JP1 23.7 mm to (24.4, 17.0), turned to 180 degrees
- moved C2 15.4 mm to (20.2, 7.62), turned to 90 degrees
- moved C1 11.3 mm to (1.84, 11.9), turned to 90 degrees
- moved IC25 0.85 mm to (8.89, 9.68), turned to 0 degrees
- moved IC3 0.85 mm to (8.89, 9.68), turned to 180 degrees
Other:
- board size 18.8 x 49 mm -> 49.1 x 18.9 mm

Commit message: planos de masa
Routing:
- added copper zone on layer 16, net GND
Changed lines of the file:
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@@
 <wire x1="0.79375" y1="14.2875" x2="0.79375" y2="16.51" width="0.4064" layer="1"/>
 <wire x1="0.79375" y1="16.51" x2="0.3175" y2="16.98625" width="0.4064" layer="1"/>
+<polygon width="0.4064" layer="16">
+<vertex x="0.15875" y="18.7325"/>
+<vertex x="48.895" y="18.7325"/>
+<vertex x="48.895" y="0.15875"/>
+<vertex x="0.15875" y="0.15875"/>
+<vertex x="0.15875" y="18.57375"/>
+</polygon>
 </signal>
 <signal name="VCC">
