File: hardware/unoedge_avillena/unoedge_v3.brd (EAGLE design)
At the start: 73.6 x 41.6 mm, 28 parts, among them IC1 74HC574D, IC2 74HC574D, IC3 74HC574D, IC4 74HC574D, IC5 74AC16245, IC6 7809, Q1 BSS123, Q2 BSS123, Q3 BSS123, Q4 BSS123

Commit message: Fallo en conexión
Connections:
- removed net N$1: Q4.2
- net EXT1: now also Q4.2
Changed lines of the file:
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@@
 <signal name="EXT1">
 <contactref element="JP1" pad="2"/>
+<contactref element="Q4" pad="2"/>
+<wire x1="5.08" y1="7.62" x2="34.12875" y2="21.76" width="0" layer="19" extent="1-1"/>
 </signal>
 <signal name="VCCIN">
@@
 <wire x1="2.54" y1="7.62" x2="64.1375" y2="19.52625" width="0" layer="19" extent="1-1"/>
 </signal>
-<signal name="N$1">
-<contactref element="Q4" pad="2"/>
-</signal>
 <signal name="+12V">
