File: hardware/unoedge_avillena/unoedge_v3.sch (EAGLE design)
At the start: 28 parts, among them IC1 74HC574D, IC2 74HC574D, IC3 74HC574D, IC4 74HC574D, IC5 74AC16245, IC6 7809, Q1 BSS123, Q2 BSS123, Q3 BSS123, Q4 BSS123

Commit message: Fallo en conexión
Connections:
- removed net N$1: Q4.S
- net EXT1: now also Q4.S
Changed lines of the file:
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@@
 </segment>
 <segment>
-<wire x1="55.88" y1="152.4" x2="45.72" y2="152.4" width="0.1524" layer="91"/>
-<label x="45.72" y="152.4" size="1.778" layer="95"/>
+<pinref part="Q4" gate="G$1" pin="S"/>
+<wire x1="50.8" y1="152.4" x2="60.96" y2="152.4" width="0.1524" layer="91"/>
+<label x="50.8" y="152.4" size="1.778" layer="95"/>
 </segment>
 </net>
@@
 </segment>
 </net>
-<net name="N$1" class="0">
-<segment>
-<pinref part="Q4" gate="G$1" pin="S"/>
-<wire x1="55.88" y1="152.4" x2="60.96" y2="152.4" width="0.1524" layer="91"/>
-</segment>
-</net>
