File: hardware/unoedge_avillena/pasivizator.brd (EAGLE design)
At the start: 73.8 x 21.9 mm, 2 parts

Commit message: Termino pasivizators
Routing:
- net N$33: track 0.00 -> 85.9 mm
- net N$36: track 0.00 -> 84.8 mm
- net N$31: track 0.00 -> 83.3 mm
- net N$37: track 0.00 -> 80.7 mm
- net N$34: track 0.00 -> 79.6 mm
- net N$4: track 0.00 -> 77.9 mm
- net N$35: track 0.00 -> 75.4 mm
- net N$20: track 0.00 -> 74.2 mm
- net N$16: track 0.00 -> 72.6 mm
- net N$46: track 0.00 -> 70.0 mm
- net N$21: track 0.00 -> 68.9 mm
- net N$26: track 0.00 -> 67.1 mm
- net N$50: track 0.00 -> 64.6 mm
- net N$47: track 0.00 -> 62.1 mm
- net N$27: track 0.00 -> 61.6 mm
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