File: hardware/otros/interface2/cartucho_throwhole.sch (EAGLE design)
At the start: 10 parts, among them IC1 74HC164N, IC2 AM29F010S, IC3 74HC32N

Commit message: 
Parts:
- removed IC2: AM29F010S, am29-memory:AM29F010S
- added U1: AM29F040S, am29-memory:AM29F040S
Connections:
- net A0: now also U1G$1.A0; no longer IC2G$1.A0
- net A1: now also U1G$1.A1; no longer IC2G$1.A1
- net A10: now also U1G$1.A10; no longer IC2G$1.A10
- net A11: now also U1G$1.A11; no longer IC2G$1.A11
- net A12: now also U1G$1.A12; no longer IC2G$1.A12
- net A13: now also U1G$1.A13; no longer IC2G$1.A13
- net A2: now also U1G$1.A2; no longer IC2G$1.A2
- net A3: now also U1G$1.A3; no longer IC2G$1.A3
- net A4: now also U1G$1.A4; no longer IC2G$1.A4
- net A5: now also U1G$1.A5; no longer IC2G$1.A5
- net A6: now also U1G$1.A6; no longer IC2G$1.A6
- net A7: now also U1G$1.A7; no longer IC2G$1.A7
- net A8: now also U1G$1.A8; no longer IC2G$1.A8
- net A9: now also U1G$1.A9; no longer IC2G$1.A9
- net CS: now also U1G$1.!CE; no longer IC2G$1.!CE
- net D0: now also U1G$1.O0; no longer IC2G$1.O0
- net D1: now also U1G$1.O1; no longer IC2G$1.O1
- net D2: now also U1G$1.O2; no longer IC2G$1.O2
- net D3: now also U1G$1.O3; no longer IC2G$1.O3
- net D4: now also U1G$1.O4; no longer IC2G$1.O4
- net D5: now also U1G$1.O5; no longer IC2G$1.O5
- net D6: now also U1G$1.O6; no longer IC2G$1.O6
- net D7: now also U1G$1.O7; no longer IC2G$1.O7
- net N$2: now also U1G$1.A18; no longer IC2G$1.A18
- net N$3: now also U1G$1.A17; no longer IC2G$1.A17
- net N$4: now also U1G$1.A16; no longer IC2G$1.A16
- net N$5: now also U1G$1.A15; no longer IC2G$1.A15
- net N$6: now also U1G$1.A14; no longer IC2G$1.A14
- net RD: now also U1G$1.!OE; no longer IC2G$1.!OE
- net WR: now also U1G$1.WE/; no longer IC2G$1.WE/

Commit message: 
Connections:
- net A14: now also IC3C.I0; no longer IC3B.I0
- net A15: now also IC3C.I1; no longer IC3B.I1
- net CS: now also IC3A.I0; no longer IC3C.I0
- net MREQ: now also IC3B.I1; no longer IC3A.I1
- net N$11: now also IC3A.O; no longer IC3C.O
- net N$7: now also IC3B.I0, IC3C.O; no longer IC3A.I0, IC3B.O
- net WR: now also IC3A.I1; no longer IC3C.I1
Other:
- moved on the sheet: IC3A, IC3B, IC3C
Changed lines of the file:
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@@
 <instance part="R1" gate="G$1" x="40.64" y="88.9" rot="R90"/>
 <instance part="S1" gate="1" x="50.8" y="73.66" rot="R180"/>
-<instance part="IC3" gate="A" x="53.34" y="17.78"/>
-<instance part="IC3" gate="B" x="25.4" y="20.32"/>
-<instance part="IC3" gate="C" x="15.24" y="63.5"/>
+<instance part="IC3" gate="B" x="53.34" y="17.78"/>
+<instance part="IC3" gate="C" x="25.4" y="20.32"/>
+<instance part="IC3" gate="A" x="15.24" y="63.5"/>
 <instance part="IC3" gate="D" x="17.78" y="43.18"/>
 <instance part="U1" gate="G$1" x="88.9" y="68.58"/>
@@
 <wire x1="10.16" y1="22.86" x2="17.78" y2="22.86" width="0.1524" layer="91"/>
 <label x="10.16" y="22.86" size="1.778" layer="95"/>
-<pinref part="IC3" gate="B" pin="I0"/>
+<pinref part="IC3" gate="C" pin="I0"/>
 </segment>
 </net>
@@
 </segment>
 <segment>
-<pinref part="IC3" gate="B" pin="I1"/>
+<pinref part="IC3" gate="C" pin="I1"/>
 <wire x1="10.16" y1="17.78" x2="17.78" y2="17.78" width="0.1524" layer="91"/>
 <label x="10.16" y="17.78" size="1.778" layer="95"/>
@@
 <wire x1="38.1" y1="15.24" x2="45.72" y2="15.24" width="0.1524" layer="91"/>
 <label x="38.1" y="15.24" size="1.778" layer="95"/>
-<pinref part="IC3" gate="A" pin="I1"/>
+<pinref part="IC3" gate="B" pin="I1"/>
 </segment>
 </net>
@@
 <wire x1="0" y1="60.96" x2="7.62" y2="60.96" width="0.1524" layer="91"/>
 <label x="0" y="60.96" size="1.778" layer="95"/>
-<pinref part="IC3" gate="C" pin="I1"/>
+<pinref part="IC3" gate="A" pin="I1"/>
 </segment>
 </net>
@@
 <wire x1="7.62" y1="53.34" x2="7.62" y2="45.72" width="0.1524" layer="91"/>
 <wire x1="7.62" y1="45.72" x2="10.16" y2="45.72" width="0.1524" layer="91"/>
-<pinref part="IC3" gate="C" pin="O"/>
+<pinref part="IC3" gate="A" pin="O"/>
 <wire x1="22.86" y1="63.5" x2="25.4" y2="63.5" width="0.1524" layer="91"/>
 </segment>
@@
 <wire x1="0" y1="66.04" x2="7.62" y2="66.04" width="0.1524" layer="91"/>
 <label x="0" y="66.04" size="1.778" layer="95"/>
-<pinref part="IC3" gate="C" pin="I0"/>
+<pinref part="IC3" gate="A" pin="I0"/>
 </segment>
 </net>
 <net name="N$7" class="0">
 <segment>
-<pinref part="IC3" gate="B" pin="O"/>
-<pinref part="IC3" gate="A" pin="I0"/>
+<pinref part="IC3" gate="C" pin="O"/>
+<pinref part="IC3" gate="B" pin="I0"/>
 <wire x1="45.72" y1="20.32" x2="33.02" y2="20.32" width="0.1524" layer="91"/>
 </segment>

Commit message: 
Connections:
- net A14: now also IC3A.I0; no longer IC3C.I0
- net A15: now also IC3A.I1; no longer IC3C.I1
- net CS: now also IC3C.I0; no longer IC3A.I0
- net N$11: now also IC3C.O; no longer IC3A.O
- net N$7: now also IC3A.O; no longer IC3C.O
- net WR: now also IC3C.I1; no longer IC3A.I1
Other:
- moved on the sheet: IC3A, IC3C
Changed lines of the file:
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@@
 <grid distance="0.1" unitdist="inch" unit="inch" style="lines" multiple="1" display="no" altdistance="0.01" altunitdist="inch" altunit="inch"/>
 <layers>
-<layer number="1" name="Top" color="4" fill="1" visible="no" active="no"/>
-<layer number="2" name="Route2" color="1" fill="3" visible="no" active="no"/>
-<layer number="3" name="Route3" color="4" fill="3" visible="no" active="no"/>
-<layer number="4" name="Route4" color="1" fill="4" visible="no" active="no"/>
-<layer number="5" name="Route5" color="4" fill="4" visible="no" active="no"/>
-<layer number="6" name="Route6" color="1" fill="8" visible="no" active="no"/>
-<layer number="7" name="Route7" color="4" fill="8" visible="no" active="no"/>
-<layer number="8" name="Route8" color="1" fill="2" visible="no" active="no"/>
-<layer number="9" name="Route9" color="4" fill="2" visible="no" active="no"/>
-<layer number="10" name="Route10" color="1" fill="7" visible="no" active="no"/>
-<layer number="11" name="Route11" color="4" fill="7" visible="no" active="no"/>
-<layer number="12" name="Route12" color="1" fill="5" visible="no" active="no"/>
-<layer number="13" name="Route13" color="4" fill="5" visible="no" active="no"/>
-<layer number="14" name="Route14" color="1" fill="6" visible="no" active="no"/>
-<layer number="15" name="Route15" color="4" fill="6" visible="no" active="no"/>
-<layer number="16" name="Bottom" color="1" fill="1" visible="no" active="no"/>
-<layer number="17" name="Pads" color="2" fill="1" visible="no" active="no"/>
-<layer number="18" name="Vias" color="2" fill="1" visible="no" active="no"/>
-<layer number="19" name="Unrouted" color="6" fill="1" visible="no" active="no"/>
-<layer number="20" name="Dimension" color="15" fill="1" visible="no" active="no"/>
-<layer number="21" name="tPlace" color="7" fill="1" visible="no" active="no"/>
-<layer number="22" name="bPlace" color="7" fill="1" visible="no" active="no"/>
-<layer number="23" name="tOrigins" color="15" fill="1" visible="no" active="no"/>
-<layer number="24" name="bOrigins" color="15" fill="1" visible="no" active="no"/>
-<layer number="25" name="tNames" color="7" fill="1" visible="no" active="no"/>
-<layer number="26" name="bNames" color="7" fill="1" visible="no" active="no"/>
-<layer number="27" name="tValues" color="7" fill="1" visible="no" active="no"/>
-<layer number="28" name="bValues" color="7" fill="1" visible="no" active="no"/>
+<layer number="1" name="Top" color="4" fill="1" visible="yes" active="no"/>
+<layer number="2" name="Route2" color="1" fill="3" visible="yes" active="no"/>
+<layer number="3" name="Route3" color="4" fill="3" visible="yes" active="no"/>
+<layer number="4" name="Route4" color="1" fill="4" visible="yes" active="no"/>
+<layer number="5" name="Route5" color="4" fill="4" visible="yes" active="no"/>
+<layer number="6" name="Route6" color="1" fill="8" visible="yes" active="no"/>
+<layer number="7" name="Route7" color="4" fill="8" visible="yes" active="no"/>
+<layer number="8" name="Route8" color="1" fill="2" visible="yes" active="no"/>
+<layer number="9" name="Route9" color="4" fill="2" visible="yes" active="no"/>
+<layer number="10" name="Route10" color="1" fill="7" visible="yes" active="no"/>
+<layer number="11" name="Route11" color="4" fill="7" visible="yes" active="no"/>
+<layer number="12" name="Route12" color="1" fill="5" visible="yes" active="no"/>
+<layer number="13" name="Route13" color="4" fill="5" visible="yes" active="no"/>
+<layer number="14" name="Route14" color="1" fill="6" visible="yes" active="no"/>
+<layer number="15" name="Route15" color="4" fill="6" visible="yes" active="no"/>
+<layer number="16" name="Bottom" color="1" fill="1" visible="yes" active="no"/>
+<layer number="17" name="Pads" color="2" fill="1" visible="yes" active="no"/>
+<layer number="18" name="Vias" color="2" fill="1" visible="yes" active="no"/>
+<layer number="19" name="Unrouted" color="6" fill="1" visible="yes" active="no"/>
+<layer number="20" name="Dimension" color="15" fill="1" visible="yes" active="no"/>
+<layer number="21" name="tPlace" color="7" fill="1" visible="yes" active="no"/>
+<layer number="22" name="bPlace" color="7" fill="1" visible="yes" active="no"/>
+<layer number="23" name="tOrigins" color="15" fill="1" visible="yes" active="no"/>
+<layer number="24" name="bOrigins" color="15" fill="1" visible="yes" active="no"/>
+<layer number="25" name="tNames" color="7" fill="1" visible="yes" active="no"/>
+<layer number="26" name="bNames" color="7" fill="1" visible="yes" active="no"/>
+<layer number="27" name="tValues" color="7" fill="1" visible="yes" active="no"/>
+<layer number="28" name="bValues" color="7" fill="1" visible="yes" active="no"/>
 <layer number="29" name="tStop" color="7" fill="3" visible="no" active="no"/>
 <layer number="30" name="bStop" color="7" fill="6" visible="no" active="no"/>
@@
 <layer number="35" name="tGlue" color="7" fill="4" visible="no" active="no"/>
 <layer number="36" name="bGlue" color="7" fill="5" visible="no" active="no"/>
-<layer number="37" name="tTest" color="7" fill="1" visible="no" active="no"/>
-<layer number="38" name="bTest" color="7" fill="1" visible="no" active="no"/>
+<layer number="37" name="tTest" color="7" fill="1" visible="yes" active="no"/>
+<layer number="38" name="bTest" color="7" fill="1" visible="yes" active="no"/>
 <layer number="39" name="tKeepout" color="4" fill="11" visible="no" active="no"/>
 <layer number="40" name="bKeepout" color="1" fill="11" visible="no" active="no"/>
@@
 <layer number="44" name="Drills" color="7" fill="1" visible="no" active="no"/>
 <layer number="45" name="Holes" color="7" fill="1" visible="no" active="no"/>
-<layer number="46" name="Milling" color="3" fill="1" visible="no" active="no"/>
-<layer number="47" name="Measures" color="7" fill="1" visible="no" active="no"/>
-<layer number="48" name="Document" color="7" fill="1" visible="no" active="no"/>
-<layer number="49" name="Reference" color="7" fill="1" visible="no" active="no"/>
-<layer number="51" name="tDocu" color="7" fill="1" visible="no" active="no"/>
-<layer number="52" name="bDocu" color="7" fill="1" visible="no" active="no"/>
+<layer number="46" name="Milling" color="3" fill="1" visible="yes" active="no"/>
+<layer number="47" name="Measures" color="7" fill="1" visible="yes" active="no"/>
+<layer number="48" name="Document" color="7" fill="1" visible="yes" active="no"/>
+<layer number="49" name="Reference" color="7" fill="1" visible="yes" active="no"/>
+<layer number="51" name="tDocu" color="7" fill="1" visible="yes" active="no"/>
+<layer number="52" name="bDocu" color="7" fill="1" visible="yes" active="no"/>
 <layer number="91" name="Nets" color="2" fill="1" visible="yes" active="yes"/>
 <layer number="92" name="Busses" color="1" fill="1" visible="yes" active="yes"/>
@@
 <instance part="S1" gate="1" x="50.8" y="73.66" rot="R180"/>
 <instance part="IC3" gate="B" x="53.34" y="17.78"/>
-<instance part="IC3" gate="C" x="25.4" y="20.32"/>
-<instance part="IC3" gate="A" x="15.24" y="63.5"/>
+<instance part="IC3" gate="A" x="25.4" y="20.32"/>
+<instance part="IC3" gate="C" x="15.24" y="63.5"/>
 <instance part="IC3" gate="D" x="17.78" y="43.18"/>
 <instance part="U1" gate="G$1" x="88.9" y="68.58"/>
@@
 <wire x1="10.16" y1="22.86" x2="17.78" y2="22.86" width="0.1524" layer="91"/>
 <label x="10.16" y="22.86" size="1.778" layer="95"/>
-<pinref part="IC3" gate="C" pin="I0"/>
+<pinref part="IC3" gate="A" pin="I0"/>
 </segment>
 </net>
@@
 </segment>
 <segment>
-<pinref part="IC3" gate="C" pin="I1"/>
+<pinref part="IC3" gate="A" pin="I1"/>
 <wire x1="10.16" y1="17.78" x2="17.78" y2="17.78" width="0.1524" layer="91"/>
 <label x="10.16" y="17.78" size="1.778" layer="95"/>
@@
 <wire x1="0" y1="60.96" x2="7.62" y2="60.96" width="0.1524" layer="91"/>
 <label x="0" y="60.96" size="1.778" layer="95"/>
-<pinref part="IC3" gate="A" pin="I1"/>
+<pinref part="IC3" gate="C" pin="I1"/>
 </segment>
 </net>
@@
 <wire x1="7.62" y1="53.34" x2="7.62" y2="45.72" width="0.1524" layer="91"/>
 <wire x1="7.62" y1="45.72" x2="10.16" y2="45.72" width="0.1524" layer="91"/>
-<pinref part="IC3" gate="A" pin="O"/>
+<pinref part="IC3" gate="C" pin="O"/>
 <wire x1="22.86" y1="63.5" x2="25.4" y2="63.5" width="0.1524" layer="91"/>
 </segment>
@@
 <wire x1="0" y1="66.04" x2="7.62" y2="66.04" width="0.1524" layer="91"/>
 <label x="0" y="66.04" size="1.778" layer="95"/>
-<pinref part="IC3" gate="A" pin="I0"/>
+<pinref part="IC3" gate="C" pin="I0"/>
 </segment>
 </net>
 <net name="N$7" class="0">
 <segment>
-<pinref part="IC3" gate="C" pin="O"/>
+<pinref part="IC3" gate="A" pin="O"/>
 <pinref part="IC3" gate="B" pin="I0"/>
 <wire x1="45.72" y1="20.32" x2="33.02" y2="20.32" width="0.1524" layer="91"/>

Commit message: 
Parts:
- removed C2: (no value), rcl:C-EU050-025X075
Connections:
- net CS: now also IC3B.O
- net GND: no longer C2.2
- net LOCK: now also IC3D.I1
- net N$11: now also IC3D.I0
- net VCC: no longer C2.1
Changed lines of the file:
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@@
 <grid distance="0.1" unitdist="inch" unit="inch" style="lines" multiple="1" display="no" altdistance="0.01" altunitdist="inch" altunit="inch"/>
 <layers>
-<layer number="1" name="Top" color="4" fill="1" visible="yes" active="no"/>
-<layer number="2" name="Route2" color="1" fill="3" visible="yes" active="no"/>
-<layer number="3" name="Route3" color="4" fill="3" visible="yes" active="no"/>
-<layer number="4" name="Route4" color="1" fill="4" visible="yes" active="no"/>
-<layer number="5" name="Route5" color="4" fill="4" visible="yes" active="no"/>
-<layer number="6" name="Route6" color="1" fill="8" visible="yes" active="no"/>
-<layer number="7" name="Route7" color="4" fill="8" visible="yes" active="no"/>
-<layer number="8" name="Route8" color="1" fill="2" visible="yes" active="no"/>
-<layer number="9" name="Route9" color="4" fill="2" visible="yes" active="no"/>
-<layer number="10" name="Route10" color="1" fill="7" visible="yes" active="no"/>
-<layer number="11" name="Route11" color="4" fill="7" visible="yes" active="no"/>
-<layer number="12" name="Route12" color="1" fill="5" visible="yes" active="no"/>
-<layer number="13" name="Route13" color="4" fill="5" visible="yes" active="no"/>
-<layer number="14" name="Route14" color="1" fill="6" visible="yes" active="no"/>
-<layer number="15" name="Route15" color="4" fill="6" visible="yes" active="no"/>
-<layer number="16" name="Bottom" color="1" fill="1" visible="yes" active="no"/>
-<layer number="17" name="Pads" color="2" fill="1" visible="yes" active="no"/>
-<layer number="18" name="Vias" color="2" fill="1" visible="yes" active="no"/>
-<layer number="19" name="Unrouted" color="6" fill="1" visible="yes" active="no"/>
-<layer number="20" name="Dimension" color="15" fill="1" visible="yes" active="no"/>
-<layer number="21" name="tPlace" color="7" fill="1" visible="yes" active="no"/>
-<layer number="22" name="bPlace" color="7" fill="1" visible="yes" active="no"/>
-<layer number="23" name="tOrigins" color="15" fill="1" visible="yes" active="no"/>
-<layer number="24" name="bOrigins" color="15" fill="1" visible="yes" active="no"/>
-<layer number="25" name="tNames" color="7" fill="1" visible="yes" active="no"/>
-<layer number="26" name="bNames" color="7" fill="1" visible="yes" active="no"/>
-<layer number="27" name="tValues" color="7" fill="1" visible="yes" active="no"/>
-<layer number="28" name="bValues" color="7" fill="1" visible="yes" active="no"/>
+<layer number="1" name="Top" color="4" fill="1" visible="no" active="no"/>
+<layer number="2" name="Route2" color="1" fill="3" visible="no" active="no"/>
+<layer number="3" name="Route3" color="4" fill="3" visible="no" active="no"/>
+<layer number="4" name="Route4" color="1" fill="4" visible="no" active="no"/>
+<layer number="5" name="Route5" color="4" fill="4" visible="no" active="no"/>
+<layer number="6" name="Route6" color="1" fill="8" visible="no" active="no"/>
+<layer number="7" name="Route7" color="4" fill="8" visible="no" active="no"/>
+<layer number="8" name="Route8" color="1" fill="2" visible="no" active="no"/>
+<layer number="9" name="Route9" color="4" fill="2" visible="no" active="no"/>
+<layer number="10" name="Route10" color="1" fill="7" visible="no" active="no"/>
+<layer number="11" name="Route11" color="4" fill="7" visible="no" active="no"/>
+<layer number="12" name="Route12" color="1" fill="5" visible="no" active="no"/>
+<layer number="13" name="Route13" color="4" fill="5" visible="no" active="no"/>
+<layer number="14" name="Route14" color="1" fill="6" visible="no" active="no"/>
+<layer number="15" name="Route15" color="4" fill="6" visible="no" active="no"/>
+<layer number="16" name="Bottom" color="1" fill="1" visible="no" active="no"/>
+<layer number="17" name="Pads" color="2" fill="1" visible="no" active="no"/>
+<layer number="18" name="Vias" color="2" fill="1" visible="no" active="no"/>
+<layer number="19" name="Unrouted" color="6" fill="1" visible="no" active="no"/>
+<layer number="20" name="Dimension" color="15" fill="1" visible="no" active="no"/>
+<layer number="21" name="tPlace" color="7" fill="1" visible="no" active="no"/>
+<layer number="22" name="bPlace" color="7" fill="1" visible="no" active="no"/>
+<layer number="23" name="tOrigins" color="15" fill="1" visible="no" active="no"/>
+<layer number="24" name="bOrigins" color="15" fill="1" visible="no" active="no"/>
+<layer number="25" name="tNames" color="7" fill="1" visible="no" active="no"/>
+<layer number="26" name="bNames" color="7" fill="1" visible="no" active="no"/>
+<layer number="27" name="tValues" color="7" fill="1" visible="no" active="no"/>
+<layer number="28" name="bValues" color="7" fill="1" visible="no" active="no"/>
 <layer number="29" name="tStop" color="7" fill="3" visible="no" active="no"/>
 <layer number="30" name="bStop" color="7" fill="6" visible="no" active="no"/>
@@
 <layer number="35" name="tGlue" color="7" fill="4" visible="no" active="no"/>
 <layer number="36" name="bGlue" color="7" fill="5" visible="no" active="no"/>
-<layer number="37" name="tTest" color="7" fill="1" visible="yes" active="no"/>
-<layer number="38" name="bTest" color="7" fill="1" visible="yes" active="no"/>
+<layer number="37" name="tTest" color="7" fill="1" visible="no" active="no"/>
+<layer number="38" name="bTest" color="7" fill="1" visible="no" active="no"/>
 <layer number="39" name="tKeepout" color="4" fill="11" visible="no" active="no"/>
 <layer number="40" name="bKeepout" color="1" fill="11" visible="no" active="no"/>
@@
 <layer number="44" name="Drills" color="7" fill="1" visible="no" active="no"/>
 <layer number="45" name="Holes" color="7" fill="1" visible="no" active="no"/>
-<layer number="46" name="Milling" color="3" fill="1" visible="yes" active="no"/>
-<layer number="47" name="Measures" color="7" fill="1" visible="yes" active="no"/>
-<layer number="48" name="Document" color="7" fill="1" visible="yes" active="no"/>
-<layer number="49" name="Reference" color="7" fill="1" visible="yes" active="no"/>
-<layer number="51" name="tDocu" color="7" fill="1" visible="yes" active="no"/>
-<layer number="52" name="bDocu" color="7" fill="1" visible="yes" active="no"/>
+<layer number="46" name="Milling" color="3" fill="1" visible="no" active="no"/>
+<layer number="47" name="Measures" color="7" fill="1" visible="no" active="no"/>
+<layer number="48" name="Document" color="7" fill="1" visible="no" active="no"/>
+<layer number="49" name="Reference" color="7" fill="1" visible="no" active="no"/>
+<layer number="51" name="tDocu" color="7" fill="1" visible="no" active="no"/>
+<layer number="52" name="bDocu" color="7" fill="1" visible="no" active="no"/>
 <layer number="91" name="Nets" color="2" fill="1" visible="yes" active="yes"/>
 <layer number="92" name="Busses" color="1" fill="1" visible="yes" active="yes"/>
@@
 <part name="C1" library="rcl" deviceset="C-EU" device="050-025X075"/>
 <part name="IC1" library="74xx-us" deviceset="74*164" device="N" technology="HC"/>
-<part name="C2" library="rcl" deviceset="C-EU" device="050-025X075"/>
 <part name="C3" library="rcl" deviceset="C-EU" device="050-025X075"/>
 <part name="C4" library="rcl" deviceset="C-EU" device="050-025X075"/>
@@
 <instance part="C1" gate="G$1" x="10.16" y="93.98"/>
 <instance part="IC1" gate="A" x="50.8" y="48.26"/>
-<instance part="C2" gate="G$1" x="17.78" y="93.98"/>
 <instance part="C3" gate="G$1" x="25.4" y="93.98"/>
 <instance part="C4" gate="G$1" x="40.64" y="76.2"/>
@@
 <pinref part="C1" gate="G$1" pin="2"/>
 <pinref part="C3" gate="G$1" pin="2"/>
-<wire x1="10.16" y1="86.36" x2="17.78" y2="86.36" width="0.1524" layer="91"/>
-<wire x1="17.78" y1="86.36" x2="25.4" y2="86.36" width="0.1524" layer="91"/>
+<wire x1="10.16" y1="86.36" x2="25.4" y2="86.36" width="0.1524" layer="91"/>
 <wire x1="25.4" y1="86.36" x2="25.4" y2="88.9" width="0.1524" layer="91"/>
-<pinref part="C2" gate="G$1" pin="2"/>
-<wire x1="17.78" y1="88.9" x2="17.78" y2="86.36" width="0.1524" layer="91"/>
 </segment>
 <segment>
@@
 <pinref part="C3" gate="G$1" pin="1"/>
 <wire x1="2.54" y1="99.06" x2="10.16" y2="99.06" width="0.1524" layer="91"/>
-<wire x1="10.16" y1="99.06" x2="17.78" y2="99.06" width="0.1524" layer="91"/>
-<wire x1="17.78" y1="99.06" x2="25.4" y2="99.06" width="0.1524" layer="91"/>
+<wire x1="10.16" y1="99.06" x2="25.4" y2="99.06" width="0.1524" layer="91"/>
 <wire x1="25.4" y1="99.06" x2="25.4" y2="96.52" width="0.1524" layer="91"/>
-<pinref part="C2" gate="G$1" pin="1"/>
-<wire x1="17.78" y1="96.52" x2="17.78" y2="99.06" width="0.1524" layer="91"/>
 <pinref part="C1" gate="G$1" pin="1"/>
 <wire x1="10.16" y1="96.52" x2="10.16" y2="99.06" width="0.1524" layer="91"/>
@@
 <pinref part="IC3" gate="C" pin="O"/>
 <wire x1="22.86" y1="63.5" x2="25.4" y2="63.5" width="0.1524" layer="91"/>
+<pinref part="IC3" gate="D" pin="I0"/>
 </segment>
 </net>
@@
 <label x="68.58" y="40.64" size="1.778" layer="95"/>
 <pinref part="U1" gate="G$1" pin="!CE"/>
+<pinref part="IC3" gate="B" pin="O"/>
 </segment>
 <segment>
@@
 <wire x1="10.16" y1="40.64" x2="2.54" y2="40.64" width="0.1524" layer="91"/>
 <label x="2.54" y="40.64" size="1.778" layer="95"/>
-</segment>
-<segment>
+<pinref part="IC3" gate="D" pin="I1"/>
+</segment>
+<segment>
