File: hardware/otros/interface2/cartucho_throwhole.sch (EAGLE design)
At the start: 9 parts, among them IC1 74HC164N, IC3 74HC32N, U1 AM29F040S

Commit message: 
Parts:
- C1, C3: value (none) -> 100nF
- C4: value (none) -> 4.7uF
- S1: value (none) -> RESET
Changed lines of the file:
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@@
 <parts>
 <part name="U$1" library="SPECTRUM" deviceset="IF2BUS" device=""/>
-<part name="C1" library="rcl" deviceset="C-EU" device="050-025X075"/>
+<part name="C1" library="rcl" deviceset="C-EU" device="050-025X075" value="100nF"/>
 <part name="IC1" library="74xx-us" deviceset="74*164" device="N" technology="HC"/>
-<part name="C3" library="rcl" deviceset="C-EU" device="050-025X075"/>
-<part name="C4" library="rcl" deviceset="C-EU" device="050-025X075"/>
+<part name="C3" library="rcl" deviceset="C-EU" device="050-025X075" value="100nF"/>
+<part name="C4" library="rcl" deviceset="C-EU" device="050-025X075" value="4.7uF"/>
 <part name="R1" library="rcl" deviceset="R-EU_" device="0204/7" value="10K"/>
-<part name="S1" library="switch-omron" deviceset="10-XX" device=""/>
+<part name="S1" library="switch-omron" deviceset="10-XX" device="" value="RESET"/>
 <part name="IC3" library="74xx-eu" deviceset="74*32" device="N" technology="HC"/>
 <part name="U1" library="am29-memory" deviceset="AM29F040S" device=""/>
+<part name="GND1" library="supply1" deviceset="GND" device=""/>
+<part name="P+1" library="supply1" deviceset="VCC" device=""/>
 </parts>
 <sheets>
@@
 <instance part="IC3" gate="D" x="17.78" y="43.18"/>
 <instance part="U1" gate="G$1" x="88.9" y="68.58"/>
+<instance part="GND1" gate="1" x="10.16" y="83.82"/>
+<instance part="P+1" gate="VCC" x="10.16" y="101.6"/>
 </instances>
 <busses>
@@
 <wire x1="38.1" y1="53.34" x2="35.56" y2="53.34" width="0.1524" layer="91"/>
 <wire x1="35.56" y1="53.34" x2="35.56" y2="55.88" width="0.1524" layer="91"/>
+<junction x="35.56" y="55.88"/>
 </segment>
 </net>
@@
 <wire x1="10.16" y1="86.36" x2="25.4" y2="86.36" width="0.1524" layer="91"/>
 <wire x1="25.4" y1="86.36" x2="25.4" y2="88.9" width="0.1524" layer="91"/>
+<junction x="10.16" y="86.36"/>
+<pinref part="GND1" gate="1" pin="GND"/>
 </segment>
 <segment>
@@
 <wire x1="48.26" y1="68.58" x2="48.26" y2="66.04" width="0.1524" layer="91"/>
 <label x="43.18" y="66.04" size="1.778" layer="95"/>
+<junction x="48.26" y="66.04"/>
 </segment>
 </net>
@@
 <wire x1="10.16" y1="96.52" x2="10.16" y2="99.06" width="0.1524" layer="91"/>
 <label x="2.54" y="99.06" size="1.778" layer="95"/>
+<junction x="10.16" y="99.06"/>
+<pinref part="P+1" gate="VCC" pin="VCC"/>
 </segment>
 </net>
@@
 <wire x1="40.64" y1="83.82" x2="40.64" y2="81.28" width="0.1524" layer="91"/>
 <label x="45.72" y="81.28" size="1.778" layer="95"/>
-</segment>
-</net>
+<junction x="48.26" y="81.28"/>
+<junction x="40.64" y="81.28"/>
+</segment>
+</net>
