File: hardware/otros/interface2/iRepair.sch (EAGLE design)
At the start: 12 parts, among them IC4 AM29F040S, IC741G332 741G3157DBVR

Commit message: Acabo iRepair
Connections:
- removed net NMI: U$3./NMI
- removed net RESET: U$3./RESET
