File: hardware/otros/comcon/comcon_version_av.sch (EAGLE design)
At the start: 101 parts, among them IC1 74LS32N, IC10 74LS365N, IC11 74LS365N, IC12 74LS365N, IC13 74LS365N, IC14 74LS365N, IC7 74LS365N, IC8 74LS365N, IC9 74LS365N

Commit message: Finalizado ruteado
Connections:
- new net N$4: IC1C.I0, IC1C.I1, IC1D.O
- net GND: no longer IC1C.I0, IC1C.I1
Changed lines of the file:
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@@
 <grid distance="0.1" unitdist="inch" unit="inch" style="lines" multiple="1" display="no" altdistance="0.01" altunitdist="inch" altunit="inch"/>
 <layers>
-<layer number="1" name="Top" color="4" fill="1" visible="yes" active="no"/>
-<layer number="2" name="Route2" color="1" fill="3" visible="yes" active="no"/>
-<layer number="3" name="Route3" color="4" fill="3" visible="yes" active="no"/>
-<layer number="4" name="Route4" color="1" fill="4" visible="yes" active="no"/>
-<layer number="5" name="Route5" color="4" fill="4" visible="yes" active="no"/>
-<layer number="6" name="Route6" color="1" fill="8" visible="yes" active="no"/>
-<layer number="7" name="Route7" color="4" fill="8" visible="yes" active="no"/>
-<layer number="8" name="Route8" color="1" fill="2" visible="yes" active="no"/>
-<layer number="9" name="Route9" color="4" fill="2" visible="yes" active="no"/>
-<layer number="10" name="Route10" color="1" fill="7" visible="yes" active="no"/>
-<layer number="11" name="Route11" color="4" fill="7" visible="yes" active="no"/>
-<layer number="12" name="Route12" color="1" fill="5" visible="yes" active="no"/>
-<layer number="13" name="Route13" color="4" fill="5" visible="yes" active="no"/>
-<layer number="14" name="Route14" color="1" fill="6" visible="yes" active="no"/>
-<layer number="15" name="Route15" color="4" fill="6" visible="yes" active="no"/>
-<layer number="16" name="Bottom" color="1" fill="1" visible="yes" active="no"/>
-<layer number="17" name="Pads" color="2" fill="1" visible="yes" active="no"/>
-<layer number="18" name="Vias" color="2" fill="1" visible="yes" active="no"/>
-<layer number="19" name="Unrouted" color="6" fill="1" visible="yes" active="no"/>
-<layer number="20" name="Dimension" color="15" fill="1" visible="yes" active="no"/>
-<layer number="21" name="tPlace" color="7" fill="1" visible="yes" active="no"/>
-<layer number="22" name="bPlace" color="7" fill="1" visible="yes" active="no"/>
-<layer number="23" name="tOrigins" color="15" fill="1" visible="yes" active="no"/>
-<layer number="24" name="bOrigins" color="15" fill="1" visible="yes" active="no"/>
-<layer number="25" name="tNames" color="7" fill="1" visible="yes" active="no"/>
-<layer number="26" name="bNames" color="7" fill="1" visible="yes" active="no"/>
-<layer number="27" name="tValues" color="7" fill="1" visible="yes" active="no"/>
-<layer number="28" name="bValues" color="7" fill="1" visible="yes" active="no"/>
+<layer number="1" name="Top" color="4" fill="1" visible="no" active="no"/>
+<layer number="2" name="Route2" color="1" fill="3" visible="no" active="no"/>
+<layer number="3" name="Route3" color="4" fill="3" visible="no" active="no"/>
+<layer number="4" name="Route4" color="1" fill="4" visible="no" active="no"/>
+<layer number="5" name="Route5" color="4" fill="4" visible="no" active="no"/>
+<layer number="6" name="Route6" color="1" fill="8" visible="no" active="no"/>
+<layer number="7" name="Route7" color="4" fill="8" visible="no" active="no"/>
+<layer number="8" name="Route8" color="1" fill="2" visible="no" active="no"/>
+<layer number="9" name="Route9" color="4" fill="2" visible="no" active="no"/>
+<layer number="10" name="Route10" color="1" fill="7" visible="no" active="no"/>
+<layer number="11" name="Route11" color="4" fill="7" visible="no" active="no"/>
+<layer number="12" name="Route12" color="1" fill="5" visible="no" active="no"/>
+<layer number="13" name="Route13" color="4" fill="5" visible="no" active="no"/>
+<layer number="14" name="Route14" color="1" fill="6" visible="no" active="no"/>
+<layer number="15" name="Route15" color="4" fill="6" visible="no" active="no"/>
+<layer number="16" name="Bottom" color="1" fill="1" visible="no" active="no"/>
+<layer number="17" name="Pads" color="2" fill="1" visible="no" active="no"/>
+<layer number="18" name="Vias" color="2" fill="1" visible="no" active="no"/>
+<layer number="19" name="Unrouted" color="6" fill="1" visible="no" active="no"/>
+<layer number="20" name="Dimension" color="15" fill="1" visible="no" active="no"/>
+<layer number="21" name="tPlace" color="7" fill="1" visible="no" active="no"/>
+<layer number="22" name="bPlace" color="7" fill="1" visible="no" active="no"/>
+<layer number="23" name="tOrigins" color="15" fill="1" visible="no" active="no"/>
+<layer number="24" name="bOrigins" color="15" fill="1" visible="no" active="no"/>
+<layer number="25" name="tNames" color="7" fill="1" visible="no" active="no"/>
+<layer number="26" name="bNames" color="7" fill="1" visible="no" active="no"/>
+<layer number="27" name="tValues" color="7" fill="1" visible="no" active="no"/>
+<layer number="28" name="bValues" color="7" fill="1" visible="no" active="no"/>
 <layer number="29" name="tStop" color="7" fill="3" visible="no" active="no"/>
 <layer number="30" name="bStop" color="7" fill="6" visible="no" active="no"/>
@@
 <layer number="35" name="tGlue" color="7" fill="4" visible="no" active="no"/>
 <layer number="36" name="bGlue" color="7" fill="5" visible="no" active="no"/>
-<layer number="37" name="tTest" color="7" fill="1" visible="yes" active="no"/>
-<layer number="38" name="bTest" color="7" fill="1" visible="yes" active="no"/>
+<layer number="37" name="tTest" color="7" fill="1" visible="no" active="no"/>
+<layer number="38" name="bTest" color="7" fill="1" visible="no" active="no"/>
 <layer number="39" name="tKeepout" color="4" fill="11" visible="no" active="no"/>
 <layer number="40" name="bKeepout" color="1" fill="11" visible="no" active="no"/>
@@
 <layer number="44" name="Drills" color="7" fill="1" visible="no" active="no"/>
 <layer number="45" name="Holes" color="7" fill="1" visible="no" active="no"/>
-<layer number="46" name="Milling" color="3" fill="1" visible="yes" active="no"/>
-<layer number="47" name="Measures" color="7" fill="1" visible="yes" active="no"/>
-<layer number="48" name="Document" color="7" fill="1" visible="yes" active="no"/>
-<layer number="49" name="Reference" color="7" fill="1" visible="yes" active="no"/>
-<layer number="50" name="dxf" color="7" fill="1" visible="yes" active="no"/>
-<layer number="51" name="tDocu" color="7" fill="1" visible="yes" active="no"/>
-<layer number="52" name="bDocu" color="7" fill="1" visible="yes" active="no"/>
-<layer number="53" name="tGND_GNDA" color="7" fill="9" visible="yes" active="no"/>
-<layer number="54" name="bGND_GNDA" color="1" fill="9" visible="yes" active="no"/>
-<layer number="56" name="wert" color="7" fill="1" visible="yes" active="no"/>
-<layer number="57" name="tCAD" color="7" fill="1" visible="yes" active="no"/>
+<layer number="46" name="Milling" color="3" fill="1" visible="no" active="no"/>
+<layer number="47" name="Measures" color="7" fill="1" visible="no" active="no"/>
+<layer number="48" name="Document" color="7" fill="1" visible="no" active="no"/>
+<layer number="49" name="Reference" color="7" fill="1" visible="no" active="no"/>
+<layer number="50" name="dxf" color="7" fill="1" visible="no" active="no"/>
+<layer number="51" name="tDocu" color="7" fill="1" visible="no" active="no"/>
+<layer number="52" name="bDocu" color="7" fill="1" visible="no" active="no"/>
+<layer number="53" name="tGND_GNDA" color="7" fill="9" visible="no" active="no"/>
+<layer number="54" name="bGND_GNDA" color="1" fill="9" visible="no" active="no"/>
+<layer number="56" name="wert" color="7" fill="1" visible="no" active="no"/>
+<layer number="57" name="tCAD" color="7" fill="1" visible="no" active="no"/>
 <layer number="90" name="Modules" color="5" fill="1" visible="yes" active="yes"/>
 <layer number="91" name="Nets" color="2" fill="1" visible="yes" active="yes"/>
@@
 <net name="GND" class="1">
 <segment>
-<wire x1="157.48" y1="12.7" x2="157.48" y2="7.62" width="0.1524" layer="91"/>
 <pinref part="GND3" gate="1" pin="GND"/>
-<pinref part="IC1" gate="C" pin="I0"/>
-<pinref part="IC1" gate="C" pin="I1"/>
-<wire x1="157.48" y1="7.62" x2="157.48" y2="-2.54" width="0.1524" layer="91"/>
-<junction x="157.48" y="7.62"/>
 <pinref part="IC1" gate="D" pin="I0"/>
 <wire x1="157.48" y1="-2.54" x2="157.48" y2="-7.62" width="0.1524" layer="91"/>
-<junction x="157.48" y="-2.54"/>
 <pinref part="IC1" gate="D" pin="I1"/>
 <wire x1="157.48" y1="-7.62" x2="157.48" y2="-15.24" width="0.1524" layer="91"/>
@@
 </segment>
 </net>
+<net name="N$4" class="1">
+<segment>
+<pinref part="IC1" gate="C" pin="I0"/>
+<wire x1="157.48" y1="12.7" x2="157.48" y2="7.62" width="0.1524" layer="91"/>
+<pinref part="IC1" gate="C" pin="I1"/>
+<wire x1="157.48" y1="7.62" x2="157.48" y2="2.54" width="0.1524" layer="91"/>
+<junction x="157.48" y="7.62"/>
+<pinref part="IC1" gate="D" pin="O"/>
+<wire x1="157.48" y1="2.54" x2="172.72" y2="2.54" width="0.1524" layer="91"/>
+<wire x1="172.72" y1="2.54" x2="172.72" y2="-5.08" width="0.1524" layer="91"/>
+</segment>
+</net>

Commit message: Añado conectores
Parts:
- added DOWNJ1, DOWNJ2, FIREJ1, FIREJ2, LEFTJ1, LEFTJ2, PIN5J1, PIN5J2, PIN9J1, PIN9J2, RIGHTJ1, RIGHTJ2, UPJ1, UPJ2: M01PTH, SparkFun-Connectors:M01PTH
- added J1, J2: (no value), SparkFun-Connectors:DB9MALE
Connections:
- new net N$10: FIREJ1.1, J1.6
- new net N$11: J1.9, PIN9J1.1
- new net N$13: J2.1, UPJ2.1
- new net N$14: DOWNJ2.1, J2.2
- new net N$15: J2.3, LEFTJ2.1
- new net N$16: J2.4, RIGHTJ2.1
- new net N$17: J2.5, PIN5J2.1
- new net N$29: FIREJ2.1, J2.6
- new net N$30: J2.9, PIN9J2.1
- new net N$5: J1.1, UPJ1.1
- new net N$6: DOWNJ1.1, J1.2
- new net N$7: J1.3, LEFTJ1.1
- new net N$8: J1.4, RIGHTJ1.1
- new net N$9: J1.5, PIN5J1.1
- net GND: now also J1.8, J2.8
Other:
- moved on the sheet: GNDJ1, GNDJ2
Changed lines of the file:
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@@
 <part name="D39" library="diode" deviceset="1N4148" device="DO35-7" value=""/>
 <part name="D40" library="diode" deviceset="1N4148" device="DO35-7" value=""/>
+<part name="GNDJ2" library="SparkFun-Connectors" deviceset="M01" device="PTH" value=""/>
 <part name="GNDJ1" library="SparkFun-Connectors" deviceset="M01" device="PTH" value=""/>
-<part name="GNDJ2" library="SparkFun-Connectors" deviceset="M01" device="PTH" value=""/>
 <part name="C7" library="rcl" deviceset="C-EU" device="050-025X075" value="100nF"/>
 <part name="C8" library="rcl" deviceset="C-EU" device="050-025X075" value="100nF"/>
@@
 <part name="IC1" library="74xx-eu" deviceset="74*32" device="N" technology="LS"/>
 <part name="U$3" library="zx_edge" deviceset="ZXSP_ED" device="2X28_SPE"/>
+<part name="J1" library="SparkFun-Connectors" deviceset="DB9" device="MALE"/>
+<part name="LEFTJ1" library="SparkFun-Connectors" deviceset="M01" device="PTH" value=""/>
+<part name="DOWNJ1" library="SparkFun-Connectors" deviceset="M01" device="PTH" value=""/>
+<part name="UPJ1" library="SparkFun-Connectors" deviceset="M01" device="PTH" value=""/>
+<part name="RIGHTJ1" library="SparkFun-Connectors" deviceset="M01" device="PTH" value=""/>
+<part name="PIN5J1" library="SparkFun-Connectors" deviceset="M01" device="PTH" value=""/>
+<part name="FIREJ1" library="SparkFun-Connectors" deviceset="M01" device="PTH" value=""/>
+<part name="PIN9J1" library="SparkFun-Connectors" deviceset="M01" device="PTH" value=""/>
+<part name="J2" library="SparkFun-Connectors" deviceset="DB9" device="MALE"/>
+<part name="LEFTJ2" library="SparkFun-Connectors" deviceset="M01" device="PTH" value=""/>
+<part name="DOWNJ2" library="SparkFun-Connectors" deviceset="M01" device="PTH" value=""/>
+<part name="UPJ2" library="SparkFun-Connectors" deviceset="M01" device="PTH" value=""/>
+<part name="RIGHTJ2" library="SparkFun-Connectors" deviceset="M01" device="PTH" value=""/>
+<part name="PIN5J2" library="SparkFun-Connectors" deviceset="M01" device="PTH" value=""/>
+<part name="FIREJ2" library="SparkFun-Connectors" deviceset="M01" device="PTH" value=""/>
+<part name="PIN9J2" library="SparkFun-Connectors" deviceset="M01" device="PTH" value=""/>
 </parts>
 <sheets>
@@
 <instance part="D39" gate="G$1" x="134.62" y="-106.68" rot="R180"/>
 <instance part="D40" gate="G$1" x="127" y="-109.22" rot="R180"/>
-<instance part="GNDJ1" gate="G$1" x="27.94" y="147.32" rot="R180"/>
-<instance part="GNDJ2" gate="G$1" x="27.94" y="137.16" rot="R180"/>
+<instance part="GNDJ2" gate="G$1" x="223.52" y="139.7" rot="R180"/>
+<instance part="GNDJ1" gate="G$1" x="35.56" y="139.7" rot="R180"/>
 <instance part="C7" gate="G$1" x="124.46" y="142.24"/>
 <instance part="C8" gate="G$1" x="132.08" y="142.24"/>
@@
 <instance part="IC1" gate="D" x="165.1" y="-5.08"/>
 <instance part="U$3" gate="G$1" x="198.12" y="-48.26"/>
+<instance part="J1" gate="G$1" x="5.08" y="142.24"/>
+<instance part="LEFTJ1" gate="G$1" x="-25.4" y="142.24"/>
+<instance part="DOWNJ1" gate="G$1" x="-25.4" y="152.4"/>
+<instance part="UPJ1" gate="G$1" x="-25.4" y="162.56"/>
+<instance part="RIGHTJ1" gate="G$1" x="-25.4" y="132.08"/>
+<instance part="PIN5J1" gate="G$1" x="-25.4" y="121.92"/>
+<instance part="FIREJ1" gate="G$1" x="35.56" y="149.86" rot="R180"/>
+<instance part="PIN9J1" gate="G$1" x="35.56" y="127" rot="R180"/>
+<instance part="J2" gate="G$1" x="193.04" y="142.24"/>
+<instance part="LEFTJ2" gate="G$1" x="162.56" y="142.24"/>
+<instance part="DOWNJ2" gate="G$1" x="162.56" y="152.4"/>
+<instance part="UPJ2" gate="G$1" x="162.56" y="162.56"/>
+<instance part="RIGHTJ2" gate="G$1" x="162.56" y="132.08"/>
+<instance part="PIN5J2" gate="G$1" x="162.56" y="121.92"/>
+<instance part="FIREJ2" gate="G$1" x="223.52" y="149.86" rot="R180"/>
+<instance part="PIN9J2" gate="G$1" x="223.52" y="127" rot="R180"/>
 </instances>
 <busses>
@@
 <segment>
 <pinref part="GNDJ1" gate="G$1" pin="1"/>
-<wire x1="12.7" y1="147.32" x2="20.32" y2="147.32" width="0.1524" layer="91"/>
-<label x="10.16" y="147.32" size="1.778" layer="95"/>
-</segment>
-<segment>
-<pinref part="GNDJ2" gate="G$1" pin="1"/>
-<wire x1="12.7" y1="137.16" x2="20.32" y2="137.16" width="0.1524" layer="91"/>
-<label x="10.16" y="137.16" size="1.778" layer="95"/>
+<label x="17.78" y="139.7" size="1.778" layer="95"/>
+<pinref part="J1" gate="G$1" pin="8"/>
+<wire x1="12.7" y1="139.7" x2="27.94" y2="139.7" width="0.1524" layer="91"/>
 </segment>
 <segment>
@@
 <pinref part="U$3" gate="G$1" pin="GND_3"/>
 <label x="187.96" y="-10.16" size="1.778" layer="95"/>
+</segment>
+<segment>
+<label x="205.74" y="139.7" size="1.778" layer="95"/>
+<pinref part="J2" gate="G$1" pin="8"/>
+<wire x1="200.66" y1="139.7" x2="215.9" y2="139.7" width="0.1524" layer="91"/>
+<pinref part="GNDJ2" gate="G$1" pin="1"/>
 </segment>
 </net>
@@
 </segment>
 </net>
+<net name="N$5" class="0">
+<segment>
+<pinref part="J1" gate="G$1" pin="1"/>
+<wire x1="-2.54" y1="147.32" x2="-12.7" y2="147.32" width="0.1524" layer="91"/>
+<pinref part="UPJ1" gate="G$1" pin="1"/>
+<wire x1="-17.78" y1="162.56" x2="-12.7" y2="162.56" width="0.1524" layer="91"/>
+<wire x1="-12.7" y1="162.56" x2="-12.7" y2="147.32" width="0.1524" layer="91"/>
+</segment>
+</net>
+<net name="N$6" class="0">
+<segment>
+<pinref part="J1" gate="G$1" pin="2"/>
+<wire x1="-2.54" y1="144.78" x2="-15.24" y2="144.78" width="0.1524" layer="91"/>
+<pinref part="DOWNJ1" gate="G$1" pin="1"/>
+<wire x1="-17.78" y1="152.4" x2="-15.24" y2="152.4" width="0.1524" layer="91"/>
+<wire x1="-15.24" y1="152.4" x2="-15.24" y2="144.78" width="0.1524" layer="91"/>
+</segment>
+</net>
+<net name="N$7" class="0">
+<segment>
+<pinref part="J1" gate="G$1" pin="3"/>
+<wire x1="-2.54" y1="142.24" x2="-17.78" y2="142.24" width="0.1524" layer="91"/>
+<pinref part="LEFTJ1" gate="G$1" pin="1"/>
+</segment>
+</net>
+<net name="N$8" class="0">
+<segment>
+<pinref part="J1" gate="G$1" pin="4"/>
+<wire x1="-2.54" y1="139.7" x2="-15.24" y2="139.7" width="0.1524" layer="91"/>
+<wire x1="-15.24" y1="139.7" x2="-15.24" y2="132.08" width="0.1524" layer="91"/>
+<pinref part="RIGHTJ1" gate="G$1" pin="1"/>
+<wire x1="-15.24" y1="132.08" x2="-17.78" y2="132.08" width="0.1524" layer="91"/>
+</segment>
+</net>
+<net name="N$9" class="0">
+<segment>
+<pinref part="J1" gate="G$1" pin="5"/>
+<wire x1="-2.54" y1="137.16" x2="-12.7" y2="137.16" width="0.1524" layer="91"/>
+<wire x1="-12.7" y1="137.16" x2="-12.7" y2="121.92" width="0.1524" layer="91"/>
+<pinref part="PIN5J1" gate="G$1" pin="1"/>
+<wire x1="-12.7" y1="121.92" x2="-17.78" y2="121.92" width="0.1524" layer="91"/>
+</segment>
+</net>
+<net name="N$10" class="0">
+<segment>
+<pinref part="J1" gate="G$1" pin="6"/>
+<wire x1="12.7" y1="144.78" x2="22.86" y2="144.78" width="0.1524" layer="91"/>
+<pinref part="FIREJ1" gate="G$1" pin="1"/>
+<wire x1="27.94" y1="149.86" x2="22.86" y2="149.86" width="0.1524" layer="91"/>
+<wire x1="22.86" y1="149.86" x2="22.86" y2="144.78" width="0.1524" layer="91"/>
+</segment>
+</net>
+<net name="N$11" class="0">
+<segment>
+<pinref part="J1" gate="G$1" pin="9"/>
+<wire x1="12.7" y1="137.16" x2="22.86" y2="137.16" width="0.1524" layer="91"/>
+<wire x1="22.86" y1="137.16" x2="22.86" y2="127" width="0.1524" layer="91"/>
+<pinref part="PIN9J1" gate="G$1" pin="1"/>
+<wire x1="22.86" y1="127" x2="27.94" y2="127" width="0.1524" layer="91"/>
+</segment>
+</net>
+<net name="N$13" class="0">
+<segment>
+<pinref part="J2" gate="G$1" pin="1"/>
+<wire x1="185.42" y1="147.32" x2="175.26" y2="147.32" width="0.1524" layer="91"/>
+<pinref part="UPJ2" gate="G$1" pin="1"/>
+<wire x1="170.18" y1="162.56" x2="175.26" y2="162.56" width="0.1524" layer="91"/>
+<wire x1="175.26" y1="162.56" x2="175.26" y2="147.32" width="0.1524" layer="91"/>
+</segment>
+</net>
+<net name="N$14" class="0">
+<segment>
+<pinref part="J2" gate="G$1" pin="2"/>
+<wire x1="185.42" y1="144.78" x2="172.72" y2="144.78" width="0.1524" layer="91"/>
+<pinref part="DOWNJ2" gate="G$1" pin="1"/>
+<wire x1="170.18" y1="152.4" x2="172.72" y2="152.4" width="0.1524" layer="91"/>
+<wire x1="172.72" y1="152.4" x2="172.72" y2="144.78" width="0.1524" layer="91"/>
+</segment>
+</net>
+<net name="N$15" class="0">
+<segment>
+<pinref part="J2" gate="G$1" pin="3"/>
+<wire x1="185.42" y1="142.24" x2="170.18" y2="142.24" width="0.1524" layer="91"/>
+<pinref part="LEFTJ2" gate="G$1" pin="1"/>
+</segment>
+</net>
+<net name="N$16" class="0">
+<segment>
+<pinref part="J2" gate="G$1" pin="4"/>
+<wire x1="185.42" y1="139.7" x2="172.72" y2="139.7" width="0.1524" layer="91"/>
+<wire x1="172.72" y1="139.7" x2="172.72" y2="132.08" width="0.1524" layer="91"/>
+<pinref part="RIGHTJ2" gate="G$1" pin="1"/>
+<wire x1="172.72" y1="132.08" x2="170.18" y2="132.08" width="0.1524" layer="91"/>
+</segment>
+</net>
+<net name="N$17" class="0">
+<segment>
+<pinref part="J2" gate="G$1" pin="5"/>
+<wire x1="185.42" y1="137.16" x2="175.26" y2="137.16" width="0.1524" layer="91"/>
+<wire x1="175.26" y1="137.16" x2="175.26" y2="121.92" width="0.1524" layer="91"/>
+<pinref part="PIN5J2" gate="G$1" pin="1"/>
+<wire x1="175.26" y1="121.92" x2="170.18" y2="121.92" width="0.1524" layer="91"/>
+</segment>
+</net>
+<net name="N$29" class="0">
+<segment>
+<pinref part="J2" gate="G$1" pin="6"/>
+<wire x1="200.66" y1="144.78" x2="210.82" y2="144.78" width="0.1524" layer="91"/>
+<pinref part="FIREJ2" gate="G$1" pin="1"/>
+<wire x1="215.9" y1="149.86" x2="210.82" y2="149.86" width="0.1524" layer="91"/>
+<wire x1="210.82" y1="149.86" x2="210.82" y2="144.78" width="0.1524" layer="91"/>
+</segment>
+</net>
+<net name="N$30" class="0">
+<segment>
+<pinref part="J2" gate="G$1" pin="9"/>
+<wire x1="200.66" y1="137.16" x2="210.82" y2="137.16" width="0.1524" layer="91"/>
+<wire x1="210.82" y1="137.16" x2="210.82" y2="127" width="0.1524" layer="91"/>
+<pinref part="PIN9J2" gate="G$1" pin="1"/>
+<wire x1="210.82" y1="127" x2="215.9" y2="127" width="0.1524" layer="91"/>
+</segment>
+</net>

Commit message: Traslado pines NMI y RESET para futuro interface
Parts:
- added GND, NMI, RESET, VCC: M01PTH, SparkFun-Connectors:M01PTH
Connections:
- new net NMI: NMI.1, U$3./NMI
- new net RESET: RESET.1, U$3./RESET
- net GND: now also GND.1
- net VCC: now also VCC.1
Changed lines of the file:
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@@
 <part name="FIREJ2" library="SparkFun-Connectors" deviceset="M01" device="PTH" value=""/>
 <part name="PIN9J2" library="SparkFun-Connectors" deviceset="M01" device="PTH" value=""/>
+<part name="GND" library="SparkFun-Connectors" deviceset="M01" device="PTH" value=""/>
+<part name="VCC" library="SparkFun-Connectors" deviceset="M01" device="PTH" value=""/>
+<part name="NMI" library="SparkFun-Connectors" deviceset="M01" device="PTH" value=""/>
+<part name="RESET" library="SparkFun-Connectors" deviceset="M01" device="PTH" value=""/>
 </parts>
 <sheets>
@@
 <instance part="FIREJ2" gate="G$1" x="223.52" y="149.86" rot="R180"/>
 <instance part="PIN9J2" gate="G$1" x="223.52" y="127" rot="R180"/>
+<instance part="GND" gate="G$1" x="81.28" y="121.92"/>
+<instance part="VCC" gate="G$1" x="81.28" y="111.76"/>
+<instance part="NMI" gate="G$1" x="116.84" y="121.92"/>
+<instance part="RESET" gate="G$1" x="116.84" y="111.76"/>
 </instances>
 <busses>
@@
 <pinref part="GNDJ2" gate="G$1" pin="1"/>
 </segment>
+<segment>
+<pinref part="GND" gate="G$1" pin="1"/>
+<wire x1="88.9" y1="121.92" x2="99.06" y2="121.92" width="0.1524" layer="91"/>
+<label x="93.98" y="121.92" size="1.778" layer="95"/>
+</segment>
 </net>
 <net name="VCC" class="1">
@@
 <label x="187.96" y="17.78" size="1.778" layer="95"/>
 </segment>
+<segment>
+<pinref part="VCC" gate="G$1" pin="1"/>
+<wire x1="88.9" y1="111.76" x2="99.06" y2="111.76" width="0.1524" layer="91"/>
+<label x="93.98" y="111.76" size="1.778" layer="95"/>
+</segment>
 </net>
 <net name="A14" class="0">
@@
 </segment>
 </net>
+<net name="RESET" class="0">
+<segment>
+<pinref part="U$3" gate="G$1" pin="/RESET"/>
+<wire x1="195.58" y1="-25.4" x2="187.96" y2="-25.4" width="0.1524" layer="91"/>
+<label x="187.96" y="-25.4" size="1.778" layer="95"/>
+</segment>
+<segment>
+<pinref part="RESET" gate="G$1" pin="1"/>
+<wire x1="124.46" y1="111.76" x2="134.62" y2="111.76" width="0.1524" layer="91"/>
+<label x="129.54" y="111.76" size="1.778" layer="95"/>
+</segment>
+</net>
+<net name="NMI" class="0">
+<segment>
+<pinref part="U$3" gate="G$1" pin="/NMI"/>
+<wire x1="195.58" y1="63.5" x2="187.96" y2="63.5" width="0.1524" layer="91"/>
+<label x="187.96" y="63.5" size="1.778" layer="95"/>
+</segment>
+<segment>
+<pinref part="NMI" gate="G$1" pin="1"/>
+<wire x1="124.46" y1="121.92" x2="134.62" y2="121.92" width="0.1524" layer="91"/>
+<label x="129.54" y="121.92" size="1.778" layer="95"/>
+</segment>
+</net>
