File: hardware/otros/zxuno2scart/adaptador_scart_v1.brd (EAGLE design)
At the start: 40.4 x 19.6 mm, 23 parts, among them Q1 BC847C, Q2 BC847C, Q3 BC847C

Commit message: 
Parts:
- Q1, Q2, Q3: value BC847C -> 2N3904
Changed lines of the file:
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@@
 <attribute name="NAME" x="9.59806875" y="12.118096875" size="0.8128" layer="25" rot="R237"/>
 </element>
-<element name="Q1" library="transistor-npn" package="SOT23" value="BC847C" x="27.6098" y="8.5344" smashed="yes" rot="MR0">
+<element name="Q1" library="transistor-npn" package="SOT23" value="2N3904" x="27.6098" y="8.5344" smashed="yes" rot="MR0">
 <attribute name="NAME" x="26.4668" y="8.6614" size="0.8128" layer="26" rot="MR0"/>
 <attribute name="VALUE" x="29.5148" y="5.3594" size="1.27" layer="28" rot="MR0"/>
 </element>
-<element name="Q2" library="transistor-npn" package="SOT23" value="BC847C" x="20.6248" y="8.4582" smashed="yes" rot="MR0">
+<element name="Q2" library="transistor-npn" package="SOT23" value="2N3904" x="20.6248" y="8.4582" smashed="yes" rot="MR0">
 <attribute name="NAME" x="21.4376" y="5.5626" size="0.8128" layer="26" rot="MR0"/>
 <attribute name="VALUE" x="22.5298" y="5.2832" size="1.27" layer="28" rot="MR0"/>
 </element>
-<element name="Q3" library="transistor-npn" package="SOT23" value="BC847C" x="13.8176" y="8.4328" smashed="yes" rot="MR0">
+<element name="Q3" library="transistor-npn" package="SOT23" value="2N3904" x="13.8176" y="8.4328" smashed="yes" rot="MR0">
 <attribute name="NAME" x="12.4206" y="9.0678" size="0.8128" layer="26" rot="MR0"/>
 <attribute name="VALUE" x="15.7226" y="5.2578" size="1.27" layer="28" rot="MR0"/>
