File: hardware/otros/teclado_sustituto_membranas/keyboard.brd (EAGLE design)
At the start: 250 x 100 mm, 98 parts, among them IC1 74HC32, IC2 74LS244DW

Commit message: 
Parts:
- moved D20 180.9 mm to (57.8, -50.5)
- moved D14 165.0 mm to (27.3, -96.8)
- moved D31 151.8 mm to (76.8, -56.2)
- moved D12 146.6 mm to (27.3, -88.6)
- moved D28 136.4 mm to (76.8, -47.9)
- moved D11 130.3 mm to (27.3, -80.3)
- moved D27 121.7 mm to (76.8, -39.7)
- moved D9 113.5 mm to (27.3, -72.1)
- moved D26 106.4 mm to (76.8, -31.4)
- moved D33 98.7 mm to (-8.57, -56.5)
- moved D6 95.8 mm to (27.3, -63.8)
- moved D5 78.5 mm to (27.3, -55.6)
- moved D4 62.7 mm to (27.3, -47.3)
- moved D19 59.4 mm to (42.9, -42.9)
- moved D3 48.4 mm to (27.3, -39.1)
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Connections:
- removed net N$91: SYMB.4, SYMB1.2
- removed net N$92: F.2, G.1
- removed net N$93: A.4, CAPS1.3
- removed net N$94: D.2, F.1
- removed net N$95: Q.2, W.1
- removed net VET: ,(COMMA).1, D2.C, JP2.8, SPACE.2
- new net N$69: SPACE.2, SYMB.1, SYMB1.1
- new net N$70: D11.A, D12.A, M.1, SYMB.2
- new net N$72: B.1, N.2
- net A10: now also T.1; no longer T.2
- net A11: now also 5.1; no longer 5.2
- net A12: now also 0.1; no longer 0.2
- net A13: now also P.1; no longer P.2
- net A15: now also ,(COMMA).1, D2.C, JP2.8, SPACE.1
- net A8: now also V.1; no longer V.2
- net A9: now also G.1; no longer G.2
- net N$10: now also B.3; no longer B.4
- net N$16: now also SYMB.4, SYMB1.3; no longer SYMB1.1
- net N$17: now also M.4; no longer M.3
- net N$18: now also C.4, D6.A; no longer J.4
- net N$19: now also B.4; no longer B.3
- net N$29: now also 3.1, 4.2; no longer 3.2, 4.1
- net N$30: now also 4.1, 5.2; no longer 4.2, 5.1
- net N$31: now also 2.1, 3.2; no longer 2.2, 3.1
- net N$32: now also 1.1, 2.2; no longer 1.2, 2.1
- net N$33: now also C.1, V.2; no longer C.2, V.1
- net N$34: now also R.1, T.2; no longer A.2, S.1
- net N$35: now also E.1; no longer T.1
- net N$36: now also W.1; no longer R.1
- net N$37: now also Q.1; no longer E.1
- net N$38: now also F.1, G.2; no longer ENTER.2, L.2
- net N$39: now also F.2; no longer S.2
- net N$40: now also D.2, S.1; no longer O.2, P.1
- net N$41: now also A.1, S.2; no longer I.2, O.1
- net N$42: now also 0.2, 9.1; no longer 6.2, 7.1
- net N$43: now also J.4; no longer C.4, D6.A
- net N$46: now also M.3; no longer M.4
- net N$52: now also SPACE.3; no longer SPACE.4
- net N$55: now also 8.1; no longer 0.1
- net N$56: now also 7.1; no longer 9.1
- net N$57: now also 6.1; no longer 8.1
- net N$58: now also C.2, X.1; no longer C.1, X.2
- net N$59: now also X.2, Z.1; no longer X.1, Z.2
- net N$60: now also CAPS.1, CAPS1.1, Z.2; no longer CAPS.2, CAPS1.2, Z.1
- net N$61: now also O.1, P.2; no longer I.1, U.2
- net N$62: now also I.1, O.2; no longer M.1, N.2
- net N$63: now also I.2, U.1; no longer K.2, L.1
- net N$64: now also U.2, Y.1; no longer U.1, Y.2
- net N$65: now also ENTER.2, L.1; no longer J.2, K.1
- net N$66: now also K.1, L.2; no longer B.2, N.1
- net N$67: now also K.2; no longer H.2
- net N$68: now also H.1, J.2; no longer SPACE.1, SYMB.2, SYMB1.3
- net N$71: now also N.1; no longer D11.A, D12.A, SYMB.1
- net N$8: now also A.4, CAPS1.3; no longer CAPS1.4
- net N$9: now also SPACE.4; no longer SPACE.3
Routing:
- net N$91: track 237.0 -> 0.00 mm
- net VET: track 181.9 -> 0.00 mm
- net N$52: track 150.7 -> 0.00 mm
- net A8: track 137.5 -> 0.00 mm
- net N$68: track 125.2 -> 0.00 mm
- net A9: track 108.2 -> 0.00 mm
- net A10: track 89.1 -> 0.00 mm
- net N$71: track 84.9 -> 0.00 mm
- net N$17: track 84.1 -> 0.00 mm
- net A11: track 77.8 -> 0.00 mm
- net N$16: track 70.3 -> 0.00 mm
- net A14: track 61.6 -> 0.00 mm
- net N$8: track 0.00 -> 61.2 mm
- net N$93: track 61.2 -> 0.00 mm
- net N$43: track 46.0 -> 0.00 mm
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
Commit message: Cambio huellas
Parts:
- removed ,(COMMA), .(PERIOD): (no value), switch-omron:B3F-40XX
- added COMMA, PERIOD: (no value), SparkFun-Electromechanical:TACTILE-SWITCH-SMD
- 0, 1, 2, 3, 4, 5, 6, 7, 8, 9, A, B, BREAK, C, CAPS, CAPS1, CAPSLOCK, D, DELETE, DOWN, E, EDIT, ENTER, EXTEND, F, G, GRAPHICS, H, I, INVV, J, K, L, LEFT, M, N, O, P, Q, QUOTES, R, RIGHT, S, SEMICOLON, SPACE, SYMB, SYMB1, T, TRUEV, U, UP, V, W, X, Y, Z: device switch-omron:B3F-40XX -> SparkFun-Electromechanical:TACTILE-SWITCH-SMD
- D1, D10, D11, D12, D13, D14, D15, D16, D17, D18, D19, D2, D20, D21, D22, D23, D24, D25, D26, D27, D28, D29, D3, D30, D31, D32, D33, D4, D5, D6, D7, D8, D9: device diode:SMC -> diode:SOD323-R
- moved BREAK 270.9 mm to (272.7, 18.1), flipped to the top
- moved SYMB 269.7 mm to (272.7, 50.5), flipped to the top, turned to 0 degrees
- moved ENTER 267.0 mm to (272.7, 72.1), flipped to the top, turned to 0 degrees
- moved L 235.2 mm to (272.7, 77.5), flipped to the top
- moved DOWN 231.8 mm to (272.7, -19.7), flipped to the top
- moved A 229.6 mm to (-33.3, -1.91), flipped to the top
- moved Q 228.9 mm to (-33.3, 52.1), flipped to the top
- moved Z 224.3 mm to (-33.3, -34.3), flipped to the top
- moved 2 219.1 mm to (-33.3, 100.6), flipped to the top
- moved K 217.3 mm to (272.7, 82.9), flipped to the top
- moved UP 215.4 mm to (272.7, -35.9), flipped to the top
- moved S 212.9 mm to (-33.3, -7.30), flipped to the top
- moved W 210.5 mm to (-33.3, 46.7), flipped to the top
- moved X 208.3 mm to (-33.3, -39.7), flipped to the top
- moved M 206.8 mm to (272.7, 55.9), flipped to the top
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Connections:
- net A10: now also T.3; no longer T.1
- net A11: now also 5.3; no longer 5.1
- net A12: now also 0.3; no longer 0.1
- net A13: now also P.3; no longer P.1
- net A14: now also ENTER.3; no longer ENTER.1
- net A15: now also COMMA.3, SPACE.3; no longer ,(COMMA).1, SPACE.1
- net A8: now also V.3; no longer V.1
- net A9: now also G.3; no longer G.1
- net CAPSLOCK: now also CAPSLOCK.3; no longer CAPSLOCK.1
- net D0: now also 1.1, EDIT.3; no longer 1.3, EDIT.1
- net D1: now also 2.1; no longer 2.3
- net D2: now also 3.1; no longer 3.3
- net D3: now also 4.1; no longer 4.3
- net D4: now also 5.1; no longer 5.3
- net DOWN: now also DOWN.3; no longer DOWN.1
- net EXTEND: now also EXTEND.3; no longer EXTEND.1
- net GND: now also CAPSLOCK.2, DOWN.2, EXTEND.2, GRAPHICS.2, INVV.2, LEFT.2, QUOTES.2, RIGHT.2, SEMICOLON.2, TRUEV.2, UP.2; no longer CAPSLOCK.4, DOWN.4, EXTEND.4, GRAPHICS.4, INVV.4, LEFT.4, QUOTES.4, RIGHT.4, SEMICOLON.4, TRUEV.4, UP.4
- net GRAPHICS: now also GRAPHICS.3; no longer GRAPHICS.1
- net INVV: now also INVV.3; no longer INVV.1
- net LEFT: now also LEFT.3; no longer LEFT.1
- net N$1: now also EDIT.2; no longer EDIT.4
- net N$10: now also B.1, H.2; no longer B.3, H.4
- net N$11: now also H.1, Y.2; no longer H.3, Y.4
- net N$12: now also 6.2, Y.1; no longer 6.4, Y.3
- net N$13: now also 2.2, W.1; no longer 2.4, W.3
- net N$14: now also S.1, W.2; no longer S.3, W.4
- net N$15: now also S.2, Z.1; no longer S.4, Z.3
- net N$16: now also SYMB.2, SYMB1.1, Z.2; no longer SYMB.4, SYMB1.3, Z.4
- net N$17: now also M.2, X.2; no longer M.4, X.4
- net N$18: now also C.2, N.2; no longer C.4, N.4
- net N$19: now also B.2, V.2; no longer B.4, V.4
- net N$2: now also EDIT.1; no longer EDIT.3
- net N$20: now also 3.2, E.1; no longer 3.4, E.3
- net N$21: now also D.1, E.2; no longer D.3, E.4
- net N$22: now also D.2, X.1; no longer D.4, X.3
- net N$23: now also 4.2, R.1; no longer 4.4, R.3
- net N$24: now also F.1, R.2; no longer F.3, R.4
- net N$25: now also C.1, F.2; no longer C.3, F.4
- net N$26: now also 5.2, T.1; no longer 5.4, T.3
- net N$27: now also G.1, T.2; no longer G.3, T.4
- net N$28: now also G.2, V.1; no longer G.4, V.3
- net N$29: now also 3.3, 4.4; no longer 3.1, 4.2
- net N$3: now also BREAK.3; no longer BREAK.1
- net N$30: now also 4.3, 5.4; no longer 4.1, 5.2
- net N$31: now also 2.3, 3.4; no longer 2.1, 3.2
- net N$32: now also 1.3, 2.4; no longer 1.1, 2.2
- net N$33: now also C.3, V.4; no longer C.1, V.2
- net N$34: now also R.3, T.4; no longer R.1, T.2
- net N$35: now also E.3, R.4; no longer E.1, R.2
- net N$36: now also E.4, W.3; no longer E.2, W.1
- net N$37: now also Q.3, W.4; no longer Q.1, W.2
- net N$38: now also F.3, G.4; no longer F.1, G.2
- net N$39: now also D.3, F.4; no longer D.1, F.2
- net N$4: now also BREAK.4; no longer BREAK.2
- net N$40: now also D.4, S.3; no longer D.2, S.1
- net N$41: now also A.3, S.4; no longer A.1, S.2
- net N$42: now also 0.4, 9.3; no longer 0.2, 9.1
- net N$43: now also J.2, N.1; no longer J.4, N.3
- net N$44: now also J.1, U.2; no longer J.3, U.4
- net N$45: now also 7.2, U.1; no longer 7.4, U.3
- net N$46: now also K.2, M.1; no longer K.4, M.3
- net N$47: now also I.2, K.1; no longer I.4, K.3
- net N$48: now also 8.2, I.1; no longer 8.4, I.3
- net N$49: now also L.2, SYMB.1; no longer L.4, SYMB.3
- net N$5: now also DELETE.3; no longer DELETE.1
- net N$50: now also L.1, O.2; no longer L.3, O.4
- net N$51: now also 9.2, O.1; no longer 9.4, O.3
- net N$52: now also ENTER.2, SPACE.1; no longer ENTER.4, SPACE.3
- net N$53: now also ENTER.1, P.2; no longer ENTER.3, P.4
- net N$54: now also 0.2, DELETE.2, P.1; no longer 0.4, DELETE.4, P.3
- net N$55: now also 8.3, 9.4; no longer 8.1, 9.2
- net N$56: now also 7.3, 8.4; no longer 7.1, 8.2
- net N$57: now also 6.3, 7.4; no longer 6.1, 7.2
- net N$58: now also C.4, X.3; no longer C.2, X.1
- net N$59: now also X.4, Z.3; no longer X.2, Z.1
- net N$6: now also 1.2, Q.1; no longer 1.4, Q.3
- net N$60: now also CAPS.3, CAPS1.3, Z.4; no longer CAPS.1, CAPS1.1, Z.2
- net N$61: now also O.3, P.4; no longer O.1, P.2
- net N$62: now also I.3, O.4; no longer I.1, O.2
- net N$63: now also I.4, U.3; no longer I.2, U.1
- net N$64: now also U.4, Y.3; no longer U.2, Y.1
- net N$65: now also ENTER.4, L.3; no longer ENTER.2, L.1
- net N$66: now also K.3, L.4; no longer K.1, L.2
- net N$67: now also J.3, K.4; no longer J.1, K.2
- net N$68: now also H.3, J.4; no longer H.1, J.2
- net N$69: now also SPACE.4, SYMB.3, SYMB1.3; no longer SPACE.2, SYMB.1, SYMB1.1
- net N$7: now also A.1, Q.2; no longer A.3, Q.4
- net N$70: now also M.3, SYMB.4; no longer M.1, SYMB.2
- net N$71: now also M.4, N.3; no longer M.2, N.1
- net N$72: now also B.3, N.4; no longer B.1, N.2
- net N$73: now also DELETE.4; no longer DELETE.2
- net N$76: now also COMMA.4, PERIOD.3; no longer ,(COMMA).2, .(PERIOD).1
- net N$78: now also COMMA.2; no longer ,(COMMA).4
- net N$79: now also PERIOD.2; no longer .(PERIOD).4
- net N$8: now also A.2, CAPS.1, CAPS1.1; no longer A.4, CAPS.3, CAPS1.3
- net N$82: now also PERIOD.1; no longer .(PERIOD).3
- net N$83: now also COMMA.1; no longer ,(COMMA).3
- net N$9: now also BREAK.2, CAPS.2, SPACE.2; no longer BREAK.4, CAPS.4, SPACE.4
- net QUOTES: now also QUOTES.3; no longer QUOTES.1
- net RIGHT: now also RIGHT.3; no longer RIGHT.1
- net SEMICOLON: now also SEMICOLON.3; no longer SEMICOLON.1
- net TRUEV: now also TRUEV.3; no longer TRUEV.1
- net UP: now also UP.3; no longer UP.1
Routing:
- net N$8: track 61.2 -> 0.00 mm
- net N$25: track 34.5 -> 0.00 mm
- net N$22: track 32.1 -> 0.00 mm
- net N$15: track 29.9 -> 0.00 mm
- net N$14: track 22.4 -> 0.00 mm
- net N$24: track 22.2 -> 0.00 mm
- net N$21: track 21.9 -> 0.00 mm
- net N$7: track 21.6 -> 0.00 mm
- net N$6: track 20.6 -> 0.00 mm
- net N$23: track 19.8 -> 0.00 mm
- net N$20: track 19.7 -> 0.00 mm
- net N$13: track 19.6 -> 0.00 mm
- net D0: track 21.0 -> 3.12 mm
- net D1: track 16.0 -> 10.8 mm
- net D3: track 40.6 -> 35.9 mm
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
Commit message: Ajuste bordes
Parts:
- moved D14 134.8 mm to (64.8, 32.7)
- moved D9 134.8 mm to (64.8, 57.5)
- moved D11 134.8 mm to (64.8, 49.2)
- moved D12 134.8 mm to (64.8, 41.0)
- moved D6 134.8 mm to (64.8, 65.7)
- moved D1 124.3 mm to (85.4, 87.3)
- moved D17 124.3 mm to (95.9, 81.0)
- moved D19 124.3 mm to (101.0, 67.0)
- moved D2 124.3 mm to (85.4, 79.1)
- moved D20 124.3 mm to (115.9, 59.4)
- moved D26 124.3 mm to (134.9, 78.4)
- moved D27 124.3 mm to (134.9, 70.2)
- moved D28 124.3 mm to (134.9, 61.9)
- moved D33 124.3 mm to (49.5, 53.3)
- moved R2 124.3 mm to (56.5, 80.3)
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
Commit message: Posicionado
Parts:
- moved SYMB 235.1 mm to (5.71, 12.1), flipped to the bottom
- moved ENTER 233.7 mm to (6.03, 59.1), flipped to the bottom
- moved BREAK 216.8 mm to (11.1, 87.9), flipped to the bottom
- moved COMMA 210.3 mm to (24.8, 11.1), flipped to the bottom
- moved L 201.0 mm to (39.1, 50.2), flipped to the bottom
- moved DOWN 186.5 mm to (43.2, 12.1), flipped to the bottom
- moved Q 185.5 mm to (194.9, 68.3), flipped to the bottom
- moved PERIOD 183.8 mm to (48.6, 30.5), flipped to the bottom
- moved K 182.7 mm to (57.8, 50.2), flipped to the bottom
- moved 2 174.0 mm to (185.4, 87.6), flipped to the bottom
- moved M 172.6 mm to (67.3, 31.4), flipped to the bottom
- moved W 167.9 mm to (175.9, 69.2), flipped to the bottom
- moved A 166.4 mm to (190.2, 49.8), flipped to the bottom
- moved UP 165.2 mm to (62.9, 12.1), flipped to the bottom
- moved J 164.5 mm to (76.8, 49.8), flipped to the bottom
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Routing:
- net D4: track 51.9 -> 0.00 mm
- net D3: track 35.9 -> 0.00 mm
- net D2: track 19.0 -> 0.00 mm
- net D1: track 10.8 -> 0.00 mm
- net D0: track 3.12 -> 0.00 mm
Other:
- board size 250 x 100 mm -> 260 x 110 mm
