File: hardware/plaquita_z80/z80.sch (EAGLE design)
At the start: 12 parts, among them U2 REG1117

Commit message: actualizo z80
Connections:
- net 3.3V renamed VCC
- removed net A11: IC1G$1.A11, J10.9
- removed net A12: IC1G$1.A12, J12.9
- removed net A13: IC1G$1.A13, J11.9
- removed net A16: J10.6
- removed net A19: J12.10
- net A0: now also IC1G$1.A15; no longer IC1G$1.A0
- net A1: now also J11.5; no longer J11.2
- net A10: now also J12.3; no longer J11.10
- net A14: now also J11.2; no longer J10.8
- net A15: now also IC1G$1.A0, J10.6; no longer IC1G$1.A15, J11.7
- net A17: now also IC1G$1.A4
- net A18: now also IC1G$1.A2
- net A2: now also IC1G$1.A13; no longer IC1G$1.A2
- net A20: now also IC1G$1.A6
- net A3: now also IC1G$1.A12; no longer IC1G$1.A3
- net A4: now also IC1G$1.A11; no longer IC1G$1.A4
- net A5: now also IC1G$1.A3; no longer IC1G$1.A5
- net A6: now also IC1G$1.A5; no longer IC1G$1.A6
- net A7: now also J12.4; no longer J10.10
- net A8: now also J11.4; no longer J11.11
- net A9: now also J10.3; no longer J12.11
- net BUSACK: now also J10.8
- net BUSREQ: now also J12.10
- net D0: now also X1.6; no longer J12.3
- net D1: now also X1.4; no longer J10.3
- net D2: now also X1.5; no longer J11.4
- net D3: now also J12.8; no longer J12.4
- net D4: now also IC1G$1.D5, J12.9; no longer IC1G$1.D4, J12.8
- net D5: now also IC1G$1.D4; no longer IC1G$1.D5
- net D6: now also J11.9; no longer J10.7
- net D7: now also X1.9; no longer J12.7
- net GND: now also X1.8
- net HALT: now also X1.1
- net INT: now also X1.3
- net IORQ: now also J10.9
- net M1: now also J12.7
- net MREQ: now also J10.10
- net NMI: now also X1.2
- net RD: now also J11.11
- net RESET: now also J10.7
- net RFSH: now also J11.7
- net WAIT: now also J11.10
- net WR: now also J12.11; no longer J11.5
